File: KiCad_Project/Wireless telemetry pcb.kicad_pcb (KiCad board)
At the start: 2 copper layers, 38.9 x 93.2 mm, 24 parts, among them J1 Conn_02x10_Counter_Clockwise, J2 Conn_02x06_Counter_Clockwise, J3 Conn_01x02_Male, Q1 BSS138, Q2 BSS138, SW1 SW_Push, U1 LD1117V33, U2 ControllerBoardV1

Commit message: Few tiny changes before ordering
Routing:
- net DIN: track 29.1 -> 29.7 mm
Other:
- board text added: "MB: J.SOL"
Changed lines of the file:
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@@
-(kicad_pcb (version 20171130) (host pcbnew "(5.1.4)-1")
+(kicad_pcb (version 20171130) (host pcbnew "(5.1.4-0-10_14)")
   (general
     (thickness 1.6)
-    (drawings 10)
-    (tracks 103)
+    (drawings 11)
+    (tracks 105)
     (zones 0)
     (modules 24)
@@
       (net 10 AD0\DIO0\CommissioningPushbutton))
   )
+  (gr_text "MB: J.SOL" (at 138.938 64.135 270) (layer B.SilkS)
+    (effects (font (size 1 1) (thickness 0.15)) (justify mirror))
+  )
   (gr_line (start 140.208 34.29) (end 140.208 115.57) (layer Edge.Cuts) (width 0.1))
   (gr_line (start 125.476 22.352) (end 140.208 34.29) (layer Edge.Cuts) (width 0.1))
@@
   (segment (start 122.541 60.198) (end 122.541 61.867) (width 0.25) (layer F.Cu) (net 1))
   (segment (start 122.541 61.867) (end 122.616 61.942) (width 0.25) (layer F.Cu) (net 1))
-  (segment (start 107.188 34.431) (end 109.65 31.969) (width 0.25) (layer F.Cu) (net 1))
-  (segment (start 109.65 31.969) (end 109.65 31.64) (width 0.25) (layer F.Cu) (net 1))
   (segment (start 107.188 46.115) (end 107.98801 45.31499) (width 0.25) (layer F.Cu) (net 1))
   (segment (start 107.98801 45.31499) (end 107.98801 35.23101) (width 0.25) (layer F.Cu) (net 1))
@@
   (segment (start 107.98801 54.53501) (end 107.687072 54.234072) (width 0.25) (layer F.Cu) (net 1))
   (segment (start 107.687072 54.234072) (end 107.188 53.735) (width 0.25) (layer F.Cu) (net 1))
+  (segment (start 109.6475 31.64) (end 109.65 31.64) (width 0.25) (layer F.Cu) (net 1))
+  (segment (start 107.188 34.0995) (end 109.6475 31.64) (width 0.25) (layer F.Cu) (net 1))
+  (segment (start 107.188 34.431) (end 107.188 34.0995) (width 0.25) (layer F.Cu) (net 1))
   (segment (start 104.267 87.884) (end 106.934 85.217) (width 0.25) (layer F.Cu) (net 2))
   (segment (start 106.934 85.217) (end 106.934 72.493) (width 0.25) (layer F.Cu) (net 2))
@@
   (segment (start 116.219 60.198) (end 116.219 61.901) (width 0.25) (layer F.Cu) (net 7))
   (segment (start 116.219 61.901) (end 116.144 61.976) (width 0.25) (layer F.Cu) (net 7))
-  (segment (start 109.65 35.64) (end 116.219 42.209) (width 0.25) (layer F.Cu) (net 7))
-  (segment (start 116.219 42.209) (end 116.219 60.198) (width 0.25) (layer F.Cu) (net 7))
+  (segment (start 116.219 41.0985) (end 116.219 60.198) (width 0.25) (layer F.Cu) (net 7))
+  (segment (start 110.7605 35.64) (end 116.219 41.0985) (width 0.25) (layer F.Cu) (net 7))
+  (segment (start 109.65 35.64) (end 110.7605 35.64) (width 0.25) (layer F.Cu) (net 7))
   (segment (start 117.094 64.076) (end 117.644 64.076) (width 0.25) (layer F.Cu) (net 8))
   (segment (start 117.644 64.076) (end 119.862 66.294) (width 0.25) (layer F.Cu) (net 8))
